Commit message: added Gazebo visualisation of the local path, and also a projector visualization

File: rosbot_description/src/rosbot_description/urdf/rosbot.xacro (robot description, xacro)
@@ -259,5 +259,5 @@
     <axis xyz="0 0 0" />
     <origin xyz="-0.03 0 0.18" rpy="0 0 0"/>
-    <parent link="body_link"/> <!-- body_link deze is aangepast ................................................................................-->
+    <parent link="body_link"/>
     <child link="camera_link"/>
   </joint>
@@ -265,5 +265,5 @@
     <collision>
       <origin xyz="0.02 0 0" rpy="0 0 0"/>
-      <geometry>0
+      <geometry>
         <box size="0.001 0.001 0.001"/>
       </geometry>
@@ -351,3 +351,31 @@
   </joint>
   <link name="range_rr"></link>
+  <!-- projector link...................................... -->
+  <joint name="projector_joint" type="fixed">
+    <axis xyz="0 0 0" />
+    <origin xyz="0.4 0 0.3" rpy="0 -0.2 0"/>
+    <parent link="body_link"/>
+    <child link="projector_link"/>
+  </joint>
+  <link name="projector_link">
+    <collision>
+      <origin xyz="0.02 0 0" rpy="0 0 0"/>
+      <geometry>
+        <box size="0.001 0.001 0.001"/>
+      </geometry>
+    </collision>
+    <visual>
+      <origin xyz="-0.01 0 -0.03" rpy="1.5707 0 1.5707"/>
+      <geometry>
+              <box size="0.001 0.001 0.001"/>
+    <!--    <mesh filename="package://rosbot_description/meshes/astra.stl" scale="0.001 0.001 0.001" /> -->
+      </geometry>
+      <material name="Black"/>
+    </visual>
+    <inertial>
+      <mass value="1e-5" />
+      <origin xyz="0 0 0" rpy="0 0 0"/>
+      <inertia ixx="0" ixy="0" ixz="0" iyy="0" iyz="0" izz="0" />
+    </inertial>
+  </link>
 </robot>

Commit message: added video capture for gazebo and AR

File: rosbot_description/src/rosbot_description/urdf/rosbot.xacro (robot description, xacro)
@@ -58,5 +58,5 @@
       <origin xyz="0 0 0.055" rpy=" 1.5707 0 1.5707"/>
       <geometry>
-        <mesh filename="package://rosbot_description/meshes/upper.stl" scale="0.001 0.001 0.001" />
+        <mesh filename="package://rosbot_description/meshes/upper.dae" scale="0.001 0.001 0.001" />
       </geometry>
       <material name="Red"/>
@@ -81,5 +81,5 @@
       <origin xyz="0 0 0" rpy="0 0 1.5707"/>
       <geometry>
-        <mesh filename="package://rosbot_description/meshes/wheel.stl" scale="0.001 0.001 0.001" />
+        <mesh filename="package://rosbot_description/meshes/wheel.dae" scale="0.001 0.001 0.001" />
       </geometry>
       <material name="Black"/>
@@ -112,5 +112,5 @@
       <origin xyz="0 0 0" rpy="0 0 -1.5707"/>
       <geometry>
-        <mesh filename="package://rosbot_description/meshes/wheel.stl" scale="0.001 0.001 0.001" />
+        <mesh filename="package://rosbot_description/meshes/wheel.dae" scale="0.001 0.001 0.001" />
       </geometry>
       <material name="Black"/>
@@ -143,5 +143,5 @@
       <origin xyz="0 0 0" rpy="0 0 1.5707"/>
       <geometry>
-        <mesh filename="package://rosbot_description/meshes/wheel.stl" scale="0.001 0.001 0.001" />
+        <mesh filename="package://rosbot_description/meshes/wheel.dae" scale="0.001 0.001 0.001" />
       </geometry>
       <material name="Black"/>
@@ -174,5 +174,5 @@
       <origin xyz="0 0 0" rpy="0 0 -1.5707"/>
       <geometry>
-        <mesh filename="package://rosbot_description/meshes/wheel.stl" scale="0.001 0.001 0.001" />
+        <mesh filename="package://rosbot_description/meshes/wheel.dae" scale="0.001 0.001 0.001" />
       </geometry>
       <material name="Black"/>
@@ -272,5 +272,5 @@
       <origin xyz="-0.01 0 -0.03" rpy="1.5707 0 1.5707"/>
       <geometry>
-        <mesh filename="package://rosbot_description/meshes/astra.stl" scale="0.001 0.001 0.001" />
+        <mesh filename="package://rosbot_description/meshes/astra.dae" scale="0.001 0.001 0.001" />
       </geometry>
       <material name="Black"/>
@@ -307,5 +307,5 @@
       <origin xyz="0 0 0" rpy="1.5707 0 4.71"/>
       <geometry>
-        <mesh filename="package://rosbot_description/meshes/rplidar.stl" scale="0.001 0.001 0.001" />
+        <mesh filename="package://rosbot_description/meshes/rplidar.dae" scale="0.001 0.001 0.001" />
       </geometry>
     </collision>
@@ -313,5 +313,5 @@
       <origin xyz="0 0 0" rpy="1.5707 0 4.71"/>
       <geometry>
-        <mesh filename="package://rosbot_description/meshes/rplidar.stl" scale="0.001 0.001 0.001" />
+        <mesh filename="package://rosbot_description/meshes/rplidar.dae" scale="0.001 0.001 0.001" />
       </geometry>
       <material name="Black"/>

Commit message: all the files for the finished internship

File: rosbot_description/src/rosbot_description/urdf/rosbot.xacro (robot description, xacro)
@@ -258,5 +258,5 @@
   <joint name="astra_joint" type="fixed">
     <axis xyz="0 0 0" />
-    <origin xyz="-0.03 0 0.18" rpy="0 0 0"/>
+    <origin xyz="-0.03 0 0.18" rpy="0 0 0"/> <!-- -0.03 0 0.18 rpy 0 0 0 -->
     <parent link="body_link"/>
     <child link="camera_link"/>
@@ -264,5 +264,5 @@
   <link name="camera_link">
     <collision>
-      <origin xyz="0.02 0 0" rpy="0 0 0"/>
+      <origin xyz="0.02 0 0" rpy="0 0 0"/>  <!-- 0.02 0 0 rpy 0 0 0 -->
       <geometry>
         <box size="0.001 0.001 0.001"/>
@@ -379,3 +379,57 @@
     </inertial>
   </link>
+ <!-- extra camera links to get 3 camera's for the kademuur in meshroom test -->
+    <!-- camera 1 link -->
+ <!-- <joint name="astra1_joint" type="fixed">
+    <axis xyz="0 0 0" />
+    <origin xyz="-0.03 0 0.98" rpy="0 -0.707 0"/>
+    <parent link="body_link"/>
+    <child link="camera1_link"/>
+  </joint>
+  <link name="camera1_link">
+    <collision>
+      <origin xyz="0.02 0 0" rpy="0 0 0"/>
+      <geometry>
+        <box size="0.001 0.001 0.001"/>
+      </geometry>
+    </collision>
+    <visual>
+      <origin xyz="-0.01 0 -0.03" rpy="1.5707 0 1.5707"/>
+      <geometry>
+        <mesh filename="package://rosbot_description/meshes/astra.dae" scale="0.001 0.001 0.001" />
+      </geometry>
+      <material name="Black"/>
+    </visual>
+    <inertial>
+      <mass value="1e-5" />
+      <origin xyz="0 0 0" rpy="0 0 0"/>
+      <inertia ixx="0" ixy="0" ixz="0" iyy="0" iyz="0" izz="0" />
+    </inertial>
+  </link>
+  <joint name="astra2_joint" type="fixed">
+    <axis xyz="0 0 0" />
+    <origin xyz="-0.03 0 1.68" rpy="0 -1.57 0"/>
+    <parent link="body_link"/>
+    <child link="camera2_link"/>
+  </joint>
+  <link name="camera2_link">
+    <collision>
+      <origin xyz="0.02 0 0" rpy="0 0 0"/>
+      <geometry>
+        <box size="0.001 0.001 0.001"/>
+      </geometry>
+    </collision>
+    <visual>
+      <origin xyz="-0.01 0 -0.03" rpy="1.5707 0 1.5707"/>
+      <geometry>
+        <mesh filename="package://rosbot_description/meshes/astra.dae" scale="0.001 0.001 0.001" />
+      </geometry>
+      <material name="Black"/>
+    </visual>
+    <inertial>
+      <mass value="1e-5" />
+      <origin xyz="0 0 0" rpy="0 0 0"/>
+      <inertia ixx="0" ixy="0" ixz="0" iyy="0" iyz="0" izz="0" />
+    </inertial>
+  </link> -->
 </robot>
